File: Electronic boards/core-controller/core-controller.sch (EAGLE design)
At the start: 15 parts, among them IC1 ATMEGA88-THIN

Commit message: Created folder for First Prototype and updated Core Controller board (with dc driver in itself, hence dc driver board is no more)
Parts:
- removed LOAD-CELL-AMP, MOTOR-DRIVER: (no value), SparkFun-Connectors:CONN_021X02_NO_SILK
- added 9V1, DC-OUT1: TERM-1X02-FABLAB, fab:TERM-1X02-FABLAB
- added AMP-CONN: (no value), SparkFun-Connectors:CONN_041X04_NO_SILK
- added AMP-GND: (no value), SparkFun-Connectors:CONN_01PTH_NO_SILK_YES_STOP
- added C4: 10uf, fab:CAP-UNPOLARIZEDFAB
- added C5: 1uf, fab:CAP-UNPOLARIZEDFAB
- added U$2: A4953, fab:A4953-H-BRIDGE-MOTOR-DRIVER
Connections:
- new net OUT1: DC-OUT1.2, U$2.OUT1
- new net OUT2: DC-OUT1.1, U$2.OUT2
- new net VDD: 9V1.2, C4.2, C5.2, U$2.VBB
- net 5V: now also AMP-CONN.1, AMP-CONN.2, IC1.VCC@2, U$2.VREF
- net CLK: now also AMP-CONN.4; no longer LOAD-CELL-AMP.2
- net DAT: now also AMP-CONN.3; no longer LOAD-CELL-AMP.1
- net DC-IN-1: now also U$2.IN1; no longer MOTOR-DRIVER.1
- net DC-IN-2: now also U$2.IN2; no longer MOTOR-DRIVER.2
- net GND: now also 9V1.1, AMP-GND.1, C4.1, C5.1, U$2.GND, U$2.LSS
Other:
- moved on the sheet: LED, R2
