File: Electronic boards/power-supply/power-supply.brd (EAGLE design)
At the start: 100 x 80 mm, 8 parts

Commit message: Updated sevaral things: blocks and structure designs, electronic boards, usability of the product, etc.
Parts:
- moved 9V-CONN2 53.5 mm to (37.1, 9.40), turned to 270 degrees
- moved 5V-CONN2 36.7 mm to (37.0, 18.1), turned to 270 degrees
- moved 5V-CONN4 24.3 mm to (37.0, 27.4), turned to 270 degrees
Routing:
- net 9V: track 32.6 -> 80.8 mm
- net 5V: track 50.8 -> 64.3 mm
Other:
- outline, holes or cut-outs redrawn
